Commit message: Added hokuyo

File: turtlebot_description/urdf/turtlebot_common_library.urdf.xacro (robot description, xacro)
@@ -7,3 +7,5 @@
   <xacro:include filename="$(find turtlebot_description)/urdf/common_properties.urdf.xacro"/>
   <xacro:include filename="$(find turtlebot_description)/urdf/turtlebot_properties.urdf.xacro"/>
+  <!--  Hokuyo Laser Sensor-->
+  <xacro:include filename="$(find turtlebot_description)/urdf/sensors/hokuyo.urdf.xacro"/>
 </robot>

File: turtlebot_description/urdf/turtlebot_gazebo.urdf.xacro (robot description, xacro)
@@ -40,3 +40,43 @@
     </gazebo>
   </xacro:macro>
+  <xacro:macro name="turtlebot_sim_laser_range_finder">
+    <!-- ULM-30LX Hokuyo Laser Range Finder -->
+    <gazebo reference="hokuyo_link">
+      <!-- <sensor type="gpu_ray" name="head_hokuyo_sensor"> -->
+        <sensor type="ray" name="head_hokuyo_sensor">
+        <pose>0 0 0 0 0 0</pose>
+        <visualize>true</visualize>
+        <update_rate>40</update_rate>
+        <ray>
+          <scan>
+            <horizontal>
+              <samples>1080</samples>
+              <resolution>0.25</resolution>
+              <min_angle>-2.3561945</min_angle>
+              <max_angle>2.3561945</max_angle>
+            </horizontal>
+          </scan>
+          <range>
+            <min>0.10</min>
+            <max>30.0</max>
+            <resolution>0.01</resolution>
+          </range>
+          <noise>
+            <type>gaussian</type>
+            <!-- Noise parameters based on published spec for Hokuyo laser
+                 achieving "+-30mm" accuracy at range < 10m.  A mean of 0.0m and
+                 stddev of 0.01m will put 99.7% of samples within 0.03m of the true
+                 reading. -->
+            <mean>0.0</mean>
+            <stddev>0.01</stddev>
+          </noise>
+        </ray>
+        <!-- <plugin name="gazebo_ros_head_hokuyo_controller" filename="libgazebo_ros_gpu_laser.so"> -->
+	  <plugin name="gazebo_ros_head_hokuyo_controller" filename="libgazebo_ros_laser.so">
+          <topicName>laserscan</topicName>
+          <frameName>hokuyo_link</frameName>
+        </plugin>
+      </sensor>
+    </gazebo>
+  </xacro:macro>
 </robot>
